Commit message: change urdf

File: aubo_description/urdf/aubo_i5.urdf (robot description, URDF)
Before this commit: robot aubo_i5, 15 links, 14 joints
Links:
- added link car_cube_link, mass 31.8228891222604; collision mesh filename=package://aubo_description/meshes/car/car_cube_link.STL; visual mesh filename=package://aubo_description/meshes/car/car_cube_link.STL
- added link kinect2_rgb_optical_frame
- added link mynt_camera_link
- link dh_grasp_link: geometry collision box size=0.15 0.05 0.15; visual box size=0.15 0.05 0.10
Joints:
- removed joint car_joint
- added joint car_base_joint: type fixed, parent base_footprint, child car_base_link, origin xyz=0.0 0.24 0.03 rpy=0.0 0.0 0.0, axis 0 0 1, limit lower=0 upper=0 effort=0 velocity=0
- added joint car_cube_joint: type fixed, parent base_footprint, child car_cube_link, origin xyz=0.35 -0.557 -0.2105 rpy=0.0 0.0 3.1415926, axis 0 0 1, limit lower=0 upper=0 effort=0 velocity=0
- added joint kinect2_rgb_optical_joint: type fixed, parent wrist3_Link, child kinect2_rgb_optical_frame, origin xyz=-0.106744813734 0.092974366887 0.0530513667371 rpy=0.179298499038  0.00762563591405 -3.12110595845, axis 0 0 1, limit lower=0 upper=0 effort=0 velocity=0
- added joint mynt_camera_joint: type fixed, parent car_base_link, child mynt_camera_link, origin xyz=0.0 0.027 0.47 rpy=-1.57 -1.57 0, axis 0 0 1, limit lower=0 upper=0 effort=0 velocity=0
- joint base_link_joint: axis (none) -> 0 0 1; limit (none) -> lower=-3.05 upper=3.05 effort=0 velocity=0; origin xyz=0.0 0.1 0.26 rpy=0.0 0.0 3.14 -> xyz=0.0 0.1 0.59 rpy=0.0 0.0 3.14
- joint dh_grasp_joint: origin xyz=0.0 -0.045 0.11 rpy=0 0 0 -> xyz=-0.02 -0.017 0.185 rpy=0 0 0; parent kinect_camera_link -> wrist3_Link
- joint wheel_left_back_joint: type revolute -> fixed
- joint wheel_left_front_joint: type revolute -> fixed
- joint wheel_right_back_joint: type revolute -> fixed
- joint wheel_right_front_joint: type revolute -> fixed

Commit message: add

File: aubo_description/urdf/aubo_i5.urdf (robot description, URDF)
Before this commit: robot aubo_i5, 18 links, 17 joints
Joints:
- joint dh_grasp_joint: origin xyz=-0.02 -0.017 0.185 rpy=0 0 0 -> xyz=0.0 0.0 0.185 rpy=0 0 0
- joint kinect2_rgb_optical_joint: origin xyz=-0.106744813734 0.092974366887 0.0530513667371 rpy=0.179298499038  0.00762563591405 -3.12110595845 -> xyz=-0.0904424697245 0.0827128670053 0.0157324730325 rpy=0.154354478521  -0.0280159632511 3.13231749676

Commit message: 修改机器人模型

File: aubo_description/urdf/aubo_i5.urdf (robot description, URDF)
Before this commit: robot aubo_i5, 18 links, 17 joints
Links:
- removed link base_footprint
- added link robot_base
Joints:
- joint base_link_joint: parent base_footprint -> robot_base
- joint car_base_joint: parent base_footprint -> robot_base
- joint car_cube_joint: parent base_footprint -> robot_base

File: aubo_description/urdf/aubo_i5.urdf.xacro (robot description, xacro)
@@ -204,7 +204,7 @@
     <limit lower="-3.05" upper="3.05" effort="0" velocity="0" />
   </joint>
-  <link name="base_footprint" />
+  <link name="robot_base" />
   <joint name="world_joint" type="fixed">
-    <parent link="base_footprint" />
+    <parent link="robot_base" />
     <child link = "base_link" />
     <origin xyz="0.0 0.0 0.6" rpy="0.0 0.0 0.0" />
